File: Hardware/LoRaWAN_SCM.kicad_sch (KiCad schematic)
At the start: 66 parts, among them J1 Conn_02x05_Odd_Even, J10 Conn_02x06_Odd_Even, J2 Conn_02x05_Odd_Even, J3 Screw_Terminal_01x02, J4 Screw_Terminal_01x03, J5 Conn_Coaxial, J6 Screw_Terminal_01x03, J7 Conn_02x06_Odd_Even, J8 Conn_02x06_Odd_Even, J9 Conn_02x06_Odd_Even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

Commit message: updated arduino code and fixed usb isuue on pcb
Parts:
- removed P1: USB_C_Plug_USB2.0, Connector_USB:USB_C_Receptacle_HRO_TYPE-C-31-M-12, symbol Connector:USB_C_Plug_USB2.0
- added J11: USB_C_Receptacle_USB2.0, symbol Connector:USB_C_Receptacle_USB2.0
Connections:
- net +5V: now also J11.A4 (VBUS), J11.A9 (VBUS), J11.B4 (VBUS), J11.B9 (VBUS)
- net D+: now also J11.A6 (D+), J11.B6 (D+)
- net D-: now also J11.A7 (D-), J11.B7 (D-)
- net GND: now also J11.A1 (GND), J11.A12 (GND), J11.B1 (GND), J11.B12 (GND), J11.S1 (SHIELD)
- net at R6.1: now also J11.B5 (CC2)
- net at R5.1: now also J11.A5 (CC1)
Changed lines of the file:
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@@
   (junction (at 307.34 86.36) (diameter 0.9144) (color 0 0 0 0))
   (junction (at 321.31 215.9) (diameter 0.9144) (color 0 0 0 0))
+  (junction (at 330.2 63.5) (diameter 0.9144) (color 0 0 0 0))
+  (junction (at 330.2 66.04) (diameter 0.9144) (color 0 0 0 0))
   (junction (at 342.9 215.9) (diameter 0.9144) (color 0 0 0 0))
   (junction (at 349.25 54.61) (diameter 0.9144) (color 0 0 0 0))
@@
     (stroke (width 0) (type solid) (color 0 0 0 0))
   )
+  (wire (pts (xy 330.2 66.04) (xy 330.2 68.58))
+    (stroke (width 0) (type solid) (color 0 0 0 0))
+  )
   (wire (pts (xy 330.2 66.04) (xy 359.41 66.04))
     (stroke (width 0) (type solid) (color 0 0 0 0))
@@
     (pin "6")
   )
-  (symbol (lib_id "Connector:USB_C_Plug_USB2.0") (at 314.96 63.5 0) (unit 1)
+  (symbol (lib_id "Connector:USB_C_Receptacle_USB2.0") (at 314.96 63.5 0) (unit 1)
     (in_bom yes) (on_board yes)
-    (property "Reference" "P1" (id 0) (at 318.77 40.64 0))
-    (property "Value" "USB_C_Plug_USB2.0" (id 1) (at 318.77 43.18 0))
-    (property "Footprint" "Connector_USB:USB_C_Receptacle_HRO_TYPE-C-31-M-12" (id 2) (at 318.77 63.5 0)
+    (property "Reference" "J11" (id 0) (at 318.77 41.91 0))
+    (property "Value" "USB_C_Receptacle_USB2.0" (id 1) (at 318.77 43.18 0))
+    (property "Footprint" "" (id 2) (at 318.77 63.5 0)
       (effects (font (size 1.27 1.27)) hide)
     )
@@
     (pin "A6")
     (pin "A7")
+    (pin "A8")
     (pin "A9")
     (pin "B1")
@@
     (pin "B4")
     (pin "B5")
+    (pin "B6")
+    (pin "B7")
+    (pin "B8")
     (pin "B9")
     (pin "S1")
@@
       (reference "J10") (unit 1) (value "Conn_02x06_Odd_Even") (footprint "Connector_PinHeader_2.54mm:PinHeader_2x06_P2.54mm_Vertical")
     )
+    (path "/9eacd668-7b1f-4281-ba64-9d9647e302e4"
+      (reference "J11") (unit 1) (value "USB_C_Receptacle_USB2.0") (footprint "")
+    )
     (path "/0c619b24-1765-4003-9401-2a4bde9b4a02"
       (reference "L1") (unit 1) (value "2.2uH") (footprint "Inductor_SMD:L_Taiyo-Yuden_NR-50xx_HandSoldering")
     )
-    (path "/92613876-daa8-4fe7-8b2c-5759e9826058"
-      (reference "P1") (unit 1) (value "USB_C_Plug_USB2.0") (footprint "Connector_USB:USB_C_Receptacle_HRO_TYPE-C-31-M-12")
-    )
     (path "/7c43e58c-e0da-467f-bf11-c38f9ef4f12d"
